Commit message: Update x1 sensor config files
Signed-off-by: wep21 <border_goldenmarket@yahoo.co.jp>

File: aip_x1_description/urdf/sensor_kit.xacro (robot description, xacro)
@@ -18,10 +18,44 @@
     <!-- lidar -->
     <xacro:VLP-16 parent="sensor_kit_base_link" name="velodyne_top" topic="/points_raw" hz="10" samples="220" gpu="$(arg gpu)">
-      <origin xyz="${calibration['sensor_kit_base_link2velodyne_top_base_link']['x']} ${calibration['sensor_kit_base_link2velodyne_top_base_link']['y']} ${calibration['sensor_kit_base_link2velodyne_top_base_link']['z']}" rpy="${calibration['sensor_kit_base_link2velodyne_top_base_link']['roll']} ${calibration['sensor_kit_base_link2velodyne_top_base_link']['pitch']} ${calibration['sensor_kit_base_link2velodyne_top_base_link']['yaw']}" />
+      <origin
+        xyz="${calibration['sensor_kit_base_link']['velodyne_top_base_link']['x']}
+             ${calibration['sensor_kit_base_link']['velodyne_top_base_link']['y']}
+             ${calibration['sensor_kit_base_link']['velodyne_top_base_link']['z']}"
+        rpy="${calibration['sensor_kit_base_link']['velodyne_top_base_link']['roll']}
+             ${calibration['sensor_kit_base_link']['velodyne_top_base_link']['pitch']}
+            ${calibration['sensor_kit_base_link']['velodyne_top_base_link']['yaw']}"
+      />
     </xacro:VLP-16>
     <xacro:include filename="$(find livox_description)/urdf/livox_horizon.xacro"/>
-    <xacro:livox_horizon_macro name="livox_front_left" parent="sensor_kit_base_link" x="${calibration['sensor_kit_base_link2livox_front_left_base_link']['x']}" y="${calibration['sensor_kit_base_link2livox_front_left_base_link']['y']}" z="${calibration['sensor_kit_base_link2livox_front_left_base_link']['z']}" roll="${calibration['sensor_kit_base_link2livox_front_left_base_link']['roll']}" pitch="${calibration['sensor_kit_base_link2livox_front_left_base_link']['pitch']}" yaw="${calibration['sensor_kit_base_link2livox_front_left_base_link']['yaw']}" />
-    <xacro:livox_horizon_macro name="livox_front_center" parent="sensor_kit_base_link" x="${calibration['sensor_kit_base_link2livox_front_center_base_link']['x']}" y="${calibration['sensor_kit_base_link2livox_front_center_base_link']['y']}" z="${calibration['sensor_kit_base_link2livox_front_center_base_link']['z']}" roll="${calibration['sensor_kit_base_link2livox_front_center_base_link']['roll']}" pitch="${calibration['sensor_kit_base_link2livox_front_center_base_link']['pitch']}" yaw="${calibration['sensor_kit_base_link2livox_front_center_base_link']['yaw']}" />
-    <xacro:livox_horizon_macro name="livox_front_right" parent="sensor_kit_base_link" x="${calibration['sensor_kit_base_link2livox_front_right_base_link']['x']}" y="${calibration['sensor_kit_base_link2livox_front_right_base_link']['y']}" z="${calibration['sensor_kit_base_link2livox_front_right_base_link']['z']}" roll="${calibration['sensor_kit_base_link2livox_front_right_base_link']['roll']}" pitch="${calibration['sensor_kit_base_link2livox_front_right_base_link']['pitch']}" yaw="${calibration['sensor_kit_base_link2livox_front_right_base_link']['yaw']}" />
+    <xacro:livox_horizon_macro
+      name="livox_front_left"
+      parent="sensor_kit_base_link"
+      x="${calibration['sensor_kit_base_link']['livox_front_left_base_link']['x']}"
+      y="${calibration['sensor_kit_base_link']['livox_front_left_base_link']['y']}"
+      z="${calibration['sensor_kit_base_link']['livox_front_left_base_link']['z']}"
+      roll="${calibration['sensor_kit_base_link']['livox_front_left_base_link']['roll']}"
+      pitch="${calibration['sensor_kit_base_link']['livox_front_left_base_link']['pitch']}"
+      yaw="${calibration['sensor_kit_base_link']['livox_front_left_base_link']['yaw']}"
+    />
+    <xacro:livox_horizon_macro
+      name="livox_front_center"
+      parent="sensor_kit_base_link"
+      x="${calibration['sensor_kit_base_link']['livox_front_center_base_link']['x']}"
+      y="${calibration['sensor_kit_base_link']['livox_front_center_base_link']['y']}"
+      z="${calibration['sensor_kit_base_link']['livox_front_center_base_link']['z']}"
+      roll="${calibration['sensor_kit_base_link']['livox_front_center_base_link']['roll']}"
+      pitch="${calibration['sensor_kit_base_link']['livox_front_center_base_link']['pitch']}"
+      yaw="${calibration['sensor_kit_base_link']['livox_front_center_base_link']['yaw']}"
+    />
+    <xacro:livox_horizon_macro
+      name="livox_front_right"
+      parent="sensor_kit_base_link"
+      x="${calibration['sensor_kit_base_link']['livox_front_right_base_link']['x']}"
+      y="${calibration['sensor_kit_base_link']['livox_front_right_base_link']['y']}"
+      z="${calibration['sensor_kit_base_link']['livox_front_right_base_link']['z']}"
+      roll="${calibration['sensor_kit_base_link']['livox_front_right_base_link']['roll']}"
+      pitch="${calibration['sensor_kit_base_link']['livox_front_right_base_link']['pitch']}"
+      yaw="${calibration['sensor_kit_base_link']['livox_front_right_base_link']['yaw']}"
+    />
   </xacro:macro>
 </robot>

File: aip_x1_description/urdf/sensors.xacro (robot description, xacro)
@@ -6,5 +6,13 @@
   <xacro:property name="calibration" value="${load_yaml('$(arg config_dir)/sensors_calibration.yaml')}"/>
   <!-- sensor kit -->
-  <xacro:sensor_kit_macro parent="base_link" x="${calibration['base_link2sensor_kit_base_link']['x']}" y="${calibration['base_link2sensor_kit_base_link']['y']}" z="${calibration['base_link2sensor_kit_base_link']['z']}" roll="${calibration['base_link2sensor_kit_base_link']['roll']}" pitch="${calibration['base_link2sensor_kit_base_link']['pitch']}" yaw="${calibration['base_link2sensor_kit_base_link']['yaw']}" />
+  <xacro:sensor_kit_macro
+    parent="base_link"
+    x="${calibration['base_link']['sensor_kit_base_link']['x']}"
+    y="${calibration['base_link']['sensor_kit_base_link']['y']}"
+    z="${calibration['base_link']['sensor_kit_base_link']['z']}"
+    roll="${calibration['base_link']['sensor_kit_base_link']['roll']}"
+    pitch="${calibration['base_link']['sensor_kit_base_link']['pitch']}"
+    yaw="${calibration['base_link']['sensor_kit_base_link']['yaw']}"
+  />
   <!-- embedded sensors -->
 </robot>
