Commit message: Update x2 sensor config files
Signed-off-by: wep21 <border_goldenmarket@yahoo.co.jp>

File: aip_x2_description/urdf/rear_unit.xacro (robot description, xacro)
@@ -19,28 +19,37 @@
     <xacro:property name="calibration" value="${load_yaml('$(arg config_dir)/rear_unit_calibration.yaml')}"/>
     <!-- BFS4(R) -->
-    <xacro:monocular_camera_macro name="camera3/camera" parent="rear_unit_base_link"
+    <xacro:monocular_camera_macro
+      name="camera3/camera"
+      parent="rear_unit_base_link"
       namespace=""
-      x="${calibration['rear_unit_base_link2camera3']['x']}"
-      y="${calibration['rear_unit_base_link2camera3']['y']}"
-      z="${calibration['rear_unit_base_link2camera3']['z']}"
-      roll="${calibration['rear_unit_base_link2camera3']['roll']}"
-      pitch="${calibration['rear_unit_base_link2camera3']['pitch']}"
-      yaw="${calibration['rear_unit_base_link2camera3']['yaw']}"
-      fps="30" width="800" height="400" fov="1.3"/>
+      x="${calibration['rear_unit_base_link']['camera3']['x']}"
+      y="${calibration['rear_unit_base_link']['camera3']['y']}"
+      z="${calibration['rear_unit_base_link']['camera3']['z']}"
+      roll="${calibration['rear_unit_base_link']['camera3']['roll']}"
+      pitch="${calibration['rear_unit_base_link']['camera3']['pitch']}"
+      yaw="${calibration['rear_unit_base_link']['camera3']['yaw']}"
+      fps="30" width="800" height="400" fov="1.3"
+    />
     <!-- lidar -->
-    <xacro:Pandar40P name="pandar_40p_rear" parent="rear_unit_base_link"
-      x="${calibration['rear_unit_base_link2pandar_40p_rear_base_link']['x']}"
-      y="${calibration['rear_unit_base_link2pandar_40p_rear_base_link']['y']}"
-      z="${calibration['rear_unit_base_link2pandar_40p_rear_base_link']['z']}"
-      roll="${calibration['rear_unit_base_link2pandar_40p_rear_base_link']['roll']}"
-      pitch="${calibration['rear_unit_base_link2pandar_40p_rear_base_link']['pitch']}"
-      yaw="${calibration['rear_unit_base_link2pandar_40p_rear_base_link']['yaw']}" />
-    <xacro:PandarQT name="pandar_qt_rear" parent="rear_unit_base_link"
-      x="${calibration['rear_unit_base_link2pandar_qt_rear_base_link']['x']}"
-      y="${calibration['rear_unit_base_link2pandar_qt_rear_base_link']['y']}"
-      z="${calibration['rear_unit_base_link2pandar_qt_rear_base_link']['z']}"
-      roll="${calibration['rear_unit_base_link2pandar_qt_rear_base_link']['roll']}"
-      pitch="${calibration['rear_unit_base_link2pandar_qt_rear_base_link']['pitch']}"
-      yaw="${calibration['rear_unit_base_link2pandar_qt_rear_base_link']['yaw']}" />
-    </xacro:macro>
+    <xacro:Pandar40P
+      name="pandar_40p_rear"
+      parent="rear_unit_base_link"
+      x="${calibration['rear_unit_base_link']['pandar_40p_rear_base_link']['x']}"
+      y="${calibration['rear_unit_base_link']['pandar_40p_rear_base_link']['y']}"
+      z="${calibration['rear_unit_base_link']['pandar_40p_rear_base_link']['z']}"
+      roll="${calibration['rear_unit_base_link']['pandar_40p_rear_base_link']['roll']}"
+      pitch="${calibration['rear_unit_base_link']['pandar_40p_rear_base_link']['pitch']}"
+      yaw="${calibration['rear_unit_base_link']['pandar_40p_rear_base_link']['yaw']}"
+    />
+    <xacro:PandarQT
+      name="pandar_qt_rear"
+      parent="rear_unit_base_link"
+      x="${calibration['rear_unit_base_link']['pandar_qt_rear_base_link']['x']}"
+      y="${calibration['rear_unit_base_link']['pandar_qt_rear_base_link']['y']}"
+      z="${calibration['rear_unit_base_link']['pandar_qt_rear_base_link']['z']}"
+      roll="${calibration['rear_unit_base_link']['pandar_qt_rear_base_link']['roll']}"
+      pitch="${calibration['rear_unit_base_link']['pandar_qt_rear_base_link']['pitch']}"
+      yaw="${calibration['rear_unit_base_link']['pandar_qt_rear_base_link']['yaw']}"
+    />
+  </xacro:macro>
 </robot>

File: aip_x2_description/urdf/sensors.xacro (robot description, xacro)
@@ -6,10 +6,34 @@
   <!-- top unit -->
   <xacro:include filename="top_unit.xacro"/>
-  <xacro:top_unit_macro parent="base_link" x="${calibration['base_link2top_unit_base_link']['x']}" y="${calibration['base_link2top_unit_base_link']['y']}" z="${calibration['base_link2top_unit_base_link']['z']}" roll="${calibration['base_link2top_unit_base_link']['roll']}" pitch="${calibration['base_link2top_unit_base_link']['pitch']}" yaw="${calibration['base_link2top_unit_base_link']['yaw']}" />
+  <xacro:top_unit_macro
+    parent="base_link"
+    x="${calibration['base_link']['top_unit_base_link']['x']}"
+    y="${calibration['base_link']['top_unit_base_link']['y']}"
+    z="${calibration['base_link']['top_unit_base_link']['z']}"
+    roll="${calibration['base_link']['top_unit_base_link']['roll']}"
+    pitch="${calibration['base_link']['top_unit_base_link']['pitch']}"
+    yaw="${calibration['base_link']['top_unit_base_link']['yaw']}"
+  />
   <!-- front unit -->
   <xacro:include filename="front_unit.xacro"/>
-  <xacro:front_unit_macro parent="base_link" x="${calibration['base_link2front_unit_base_link']['x']}" y="${calibration['base_link2front_unit_base_link']['y']}" z="${calibration['base_link2front_unit_base_link']['z']}" roll="${calibration['base_link2front_unit_base_link']['roll']}" pitch="${calibration['base_link2front_unit_base_link']['pitch']}" yaw="${calibration['base_link2front_unit_base_link']['yaw']}" />
+  <xacro:front_unit_macro
+    parent="base_link"
+    x="${calibration['base_link']['front_unit_base_link']['x']}"
+    y="${calibration['base_link']['front_unit_base_link']['y']}"
+    z="${calibration['base_link']['front_unit_base_link']['z']}"
+    roll="${calibration['base_link']['front_unit_base_link']['roll']}"
+    pitch="${calibration['base_link']['front_unit_base_link']['pitch']}"
+    yaw="${calibration['base_link']['front_unit_base_link']['yaw']}"
+  />
   <!-- rear unit -->
   <xacro:include filename="rear_unit.xacro"/>
-  <xacro:rear_unit_macro parent="base_link" x="${calibration['base_link2rear_unit_base_link']['x']}" y="${calibration['base_link2rear_unit_base_link']['y']}" z="${calibration['base_link2rear_unit_base_link']['z']}" roll="${calibration['base_link2rear_unit_base_link']['roll']}" pitch="${calibration['base_link2rear_unit_base_link']['pitch']}" yaw="${calibration['base_link2rear_unit_base_link']['yaw']}" />
+  <xacro:rear_unit_macro
+    parent="base_link"
+    x="${calibration['base_link']['rear_unit_base_link']['x']}"
+    y="${calibration['base_link']['rear_unit_base_link']['y']}"
+    z="${calibration['base_link']['rear_unit_base_link']['z']}"
+    roll="${calibration['base_link']['rear_unit_base_link']['roll']}"
+    pitch="${calibration['base_link']['rear_unit_base_link']['pitch']}"
+    yaw="${calibration['base_link']['rear_unit_base_link']['yaw']}"
+  />
 </robot>

File: aip_x2_description/urdf/top_unit.xacro (robot description, xacro)
@@ -21,48 +21,144 @@
     <!-- lidar -->
     <!-- left -->
-    <xacro:Pandar40P name="pandar_40p_left" parent="top_unit_base_link"
-      x="${calibration['top_unit_base_link2pandar_40p_left_base_link']['x']}"
-      y="${calibration['top_unit_base_link2pandar_40p_left_base_link']['y']}"
-      z="${calibration['top_unit_base_link2pandar_40p_left_base_link']['z']}"
-      roll="${calibration['top_unit_base_link2pandar_40p_left_base_link']['roll']}"
-      pitch="${calibration['top_unit_base_link2pandar_40p_left_base_link']['pitch']}"
-      yaw="${calibration['top_unit_base_link2pandar_40p_left_base_link']['yaw']}" />
-    <xacro:PandarQT name="pandar_qt_left" parent="top_unit_base_link"
-      x="${calibration['top_unit_base_link2pandar_qt_left_base_link']['x']}"
-      y="${calibration['top_unit_base_link2pandar_qt_left_base_link']['y']}"
-      z="${calibration['top_unit_base_link2pandar_qt_left_base_link']['z']}"
-      roll="${calibration['top_unit_base_link2pandar_qt_left_base_link']['roll']}"
-      pitch="${calibration['top_unit_base_link2pandar_qt_left_base_link']['pitch']}"
-      yaw="${calibration['top_unit_base_link2pandar_qt_left_base_link']['yaw']}" />
+    <xacro:Pandar40P
+      name="pandar_40p_left"
+      parent="top_unit_base_link"
+      x="${calibration['top_unit_base_link']['pandar_40p_left_base_link']['x']}"
+      y="${calibration['top_unit_base_link']['pandar_40p_left_base_link']['y']}"
+      z="${calibration['top_unit_base_link']['pandar_40p_left_base_link']['z']}"
+      roll="${calibration['top_unit_base_link']['pandar_40p_left_base_link']['roll']}"
+      pitch="${calibration['top_unit_base_link']['pandar_40p_left_base_link']['pitch']}"
+      yaw="${calibration['top_unit_base_link']['pandar_40p_left_base_link']['yaw']}"
+    />
+    <xacro:PandarQT
+      name="pandar_qt_left"
+      parent="top_unit_base_link"
+      x="${calibration['top_unit_base_link']['pandar_qt_left_base_link']['x']}"
+      y="${calibration['top_unit_base_link']['pandar_qt_left_base_link']['y']}"
+      z="${calibration['top_unit_base_link']['pandar_qt_left_base_link']['z']}"
+      roll="${calibration['top_unit_base_link']['pandar_qt_left_base_link']['roll']}"
+      pitch="${calibration['top_unit_base_link']['pandar_qt_left_base_link']['pitch']}"
+      yaw="${calibration['top_unit_base_link']['pandar_qt_left_base_link']['yaw']}"
+    />
     <!-- right -->
-    <xacro:Pandar40P name="pandar_40p_right" parent="top_unit_base_link"
-      x="${calibration['top_unit_base_link2pandar_40p_right_base_link']['x']}"
-      y="${calibration['top_unit_base_link2pandar_40p_right_base_link']['y']}"
-      z="${calibration['top_unit_base_link2pandar_40p_right_base_link']['z']}"
-      roll="${calibration['top_unit_base_link2pandar_40p_right_base_link']['roll']}"
-      pitch="${calibration['top_unit_base_link2pandar_40p_right_base_link']['pitch']}"
-      yaw="${calibration['top_unit_base_link2pandar_40p_right_base_link']['yaw']}" />
-    <xacro:PandarQT name="pandar_qt_right" parent="top_unit_base_link"
-      x="${calibration['top_unit_base_link2pandar_qt_right_base_link']['x']}"
-      y="${calibration['top_unit_base_link2pandar_qt_right_base_link']['y']}"
-      z="${calibration['top_unit_base_link2pandar_qt_right_base_link']['z']}"
-      roll="${calibration['top_unit_base_link2pandar_qt_right_base_link']['roll']}"
-      pitch="${calibration['top_unit_base_link2pandar_qt_right_base_link']['pitch']}"
-      yaw="${calibration['top_unit_base_link2pandar_qt_right_base_link']['yaw']}" />
+    <xacro:Pandar40P
+      name="pandar_40p_right"
+      parent="top_unit_base_link"
+      x="${calibration['top_unit_base_link']['pandar_40p_right_base_link']['x']}"
+      y="${calibration['top_unit_base_link']['pandar_40p_right_base_link']['y']}"
+      z="${calibration['top_unit_base_link']['pandar_40p_right_base_link']['z']}"
+      roll="${calibration['top_unit_base_link']['pandar_40p_right_base_link']['roll']}"
+      pitch="${calibration['top_unit_base_link']['pandar_40p_right_base_link']['pitch']}"
+      yaw="${calibration['top_unit_base_link']['pandar_40p_right_base_link']['yaw']}"
+    />
+    <xacro:PandarQT
+      name="pandar_qt_right"
+      parent="top_unit_base_link"
+      x="${calibration['top_unit_base_link']['pandar_qt_right_base_link']['x']}"
+      y="${calibration['top_unit_base_link']['pandar_qt_right_base_link']['y']}"
+      z="${calibration['top_unit_base_link']['pandar_qt_right_base_link']['z']}"
+      roll="${calibration['top_unit_base_link']['pandar_qt_right_base_link']['roll']}"
+      pitch="${calibration['top_unit_base_link']['pandar_qt_right_base_link']['pitch']}"
+      yaw="${calibration['top_unit_base_link']['pandar_qt_right_base_link']['yaw']}"
+    />
     <!-- camera -->
     <!-- TLR -->
-    <xacro:monocular_camera_macro name="traffic_light_camera/camera" parent="top_unit_base_link" namespace="" x="${calibration['top_unit_base_link2traffic_light_camera']['x']}" y="${calibration['top_unit_base_link2traffic_light_camera']['y']}" z="${calibration['top_unit_base_link2traffic_light_camera']['z']}" roll="${calibration['top_unit_base_link2traffic_light_camera']['roll']}" pitch="${calibration['top_unit_base_link2traffic_light_camera']['pitch']}" yaw="${calibration['top_unit_base_link2traffic_light_camera']['yaw']}" fps="30" width="800" height="400" fov="1.3"/>
+    <xacro:monocular_camera_macro
+      name="traffic_light_camera/camera"
+      parent="top_unit_base_link"
+      namespace=""
+      x="${calibration['top_unit_base_link']['traffic_light_camera']['x']}"
+      y="${calibration['top_unit_base_link']['traffic_light_camera']['y']}"
+      z="${calibration['top_unit_base_link']['traffic_light_camera']['z']}"
+      roll="${calibration['top_unit_base_link']['traffic_light_camera']['roll']}"
+      pitch="${calibration['top_unit_base_link']['traffic_light_camera']['pitch']}"
+      yaw="${calibration['top_unit_base_link']['traffic_light_camera']['yaw']}"
+      fps="30"
+      width="800"
+      height="400"
+      fov="1.3"
+    />
     <!-- BFS1(F) -->
-    <xacro:monocular_camera_macro name="camera0/camera" parent="top_unit_base_link" namespace="" x="${calibration['top_unit_base_link2camera0']['x']}" y="${calibration['top_unit_base_link2camera0']['y']}" z="${calibration['top_unit_base_link2camera0']['z']}" roll="${calibration['top_unit_base_link2camera0']['roll']}" pitch="${calibration['top_unit_base_link2camera0']['pitch']}" yaw="${calibration['top_unit_base_link2camera0']['yaw']}" fps="30" width="800" height="400" fov="1.3"/>
+    <xacro:monocular_camera_macro
+      name="camera0/camera"
+      parent="top_unit_base_link"
+      namespace=""
+      x="${calibration['top_unit_base_link']['camera0']['x']}"
+      y="${calibration['top_unit_base_link']['camera0']['y']}"
+      z="${calibration['top_unit_base_link']['camera0']['z']}"
+      roll="${calibration['top_unit_base_link']['camera0']['roll']}"
+      pitch="${calibration['top_unit_base_link']['camera0']['pitch']}"
+      yaw="${calibration['top_unit_base_link']['camera0']['yaw']}"
+      fps="30"
+      width="800"
+      height="400"
+      fov="1.3"
+    />
     <!-- BFS2(RF) -->
-    <xacro:monocular_camera_macro name="camera1/camera" parent="top_unit_base_link" namespace="" x="${calibration['top_unit_base_link2camera1']['x']}" y="${calibration['top_unit_base_link2camera1']['y']}" z="${calibration['top_unit_base_link2camera1']['z']}" roll="${calibration['top_unit_base_link2camera1']['roll']}" pitch="${calibration['top_unit_base_link2camera1']['pitch']}" yaw="${calibration['top_unit_base_link2camera1']['yaw']}" fps="30" width="800" height="400" fov="1.3"/>
+    <xacro:monocular_camera_macro
+      name="camera1/camera"
+      parent="top_unit_base_link"
+      namespace=""
+      x="${calibration['top_unit_base_link']['camera1']['x']}"
+      y="${calibration['top_unit_base_link']['camera1']['y']}"
+      z="${calibration['top_unit_base_link']['camera1']['z']}"
+      roll="${calibration['top_unit_base_link']['camera1']['roll']}"
+      pitch="${calibration['top_unit_base_link']['camera1']['pitch']}"
+      yaw="${calibration['top_unit_base_link']['camera1']['yaw']}"
+      fps="30"
+      width="800"
+      height="400"
+      fov="1.3"
+    />
     <!-- BFS3(RR) -->
-    <xacro:monocular_camera_macro name="camera2/camera" parent="top_unit_base_link" namespace="" x="${calibration['top_unit_base_link2camera2']['x']}" y="${calibration['top_unit_base_link2camera2']['y']}" z="${calibration['top_unit_base_link2camera2']['z']}" roll="${calibration['top_unit_base_link2camera2']['roll']}" pitch="${calibration['top_unit_base_link2camera2']['pitch']}" yaw="${calibration['top_unit_base_link2camera2']['yaw']}" fps="30" width="800" height="400" fov="1.3"/>
+    <xacro:monocular_camera_macro
+      name="camera2/camera"
+      parent="top_unit_base_link"
+      namespace=""
+      x="${calibration['top_unit_base_link']['camera2']['x']}"
+      y="${calibration['top_unit_base_link']['camera2']['y']}"
+      z="${calibration['top_unit_base_link']['camera2']['z']}"
+      roll="${calibration['top_unit_base_link']['camera2']['roll']}"
+      pitch="${calibration['top_unit_base_link']['camera2']['pitch']}"
+      yaw="${calibration['top_unit_base_link']['camera2']['yaw']}"
+      fps="30"
+      width="800"
+      height="400"
+      fov="1.3"
+    />
     <!-- BFS4(R) -->
     <!-- embedded! -->
     <!-- BFS5(LR) -->
-    <xacro:monocular_camera_macro name="camera4/camera" parent="top_unit_base_link" namespace="" x="${calibration['top_unit_base_link2camera4']['x']}" y="${calibration['top_unit_base_link2camera4']['y']}" z="${calibration['top_unit_base_link2camera4']['z']}" roll="${calibration['top_unit_base_link2camera4']['roll']}" pitch="${calibration['top_unit_base_link2camera4']['pitch']}" yaw="${calibration['top_unit_base_link2camera4']['yaw']}" fps="30" width="800" height="400" fov="1.3"/>
+    <xacro:monocular_camera_macro
+      name="camera4/camera"
+      parent="top_unit_base_link"
+      namespace=""
+      x="${calibration['top_unit_base_link']['camera4']['x']}"
+      y="${calibration['top_unit_base_link']['camera4']['y']}"
+      z="${calibration['top_unit_base_link']['camera4']['z']}"
+      roll="${calibration['top_unit_base_link']['camera4']['roll']}"
+      pitch="${calibration['top_unit_base_link']['camera4']['pitch']}"
+      yaw="${calibration['top_unit_base_link']['camera4']['yaw']}"
+      fps="30"
+      width="800"
+      height="400"
+      fov="1.3"
+    />
     <!-- BFS6(LR) -->
-    <xacro:monocular_camera_macro name="camera5/camera" parent="top_unit_base_link" namespace="" x="${calibration['top_unit_base_link2camera5']['x']}" y="${calibration['top_unit_base_link2camera5']['y']}" z="${calibration['top_unit_base_link2camera5']['z']}" roll="${calibration['top_unit_base_link2camera5']['roll']}" pitch="${calibration['top_unit_base_link2camera5']['pitch']}" yaw="${calibration['top_unit_base_link2camera5']['yaw']}" fps="30" width="800" height="400" fov="1.3"/>
+    <xacro:monocular_camera_macro
+      name="camera5/camera"
+      parent="top_unit_base_link"
+      namespace=""
+      x="${calibration['top_unit_base_link']['camera5']['x']}"
+      y="${calibration['top_unit_base_link']['camera5']['y']}"
+      z="${calibration['top_unit_base_link']['camera5']['z']}"
+      roll="${calibration['top_unit_base_link']['camera5']['roll']}"
+      pitch="${calibration['top_unit_base_link']['camera5']['pitch']}"
+      yaw="${calibration['top_unit_base_link']['camera5']['yaw']}"
+      fps="30"
+      width="800"
+      height="400"
+      fov="1.3"
+    />
     <!-- gnss -->
     <!-- left -->
@@ -71,11 +167,12 @@
       parent="top_unit_base_link"
       namespace=""
-      x="${calibration['top_unit_base_link2gnss_right']['x']}"
-      y="${calibration['top_unit_base_link2gnss_right']['y']}"
-      z="${calibration['top_unit_base_link2gnss_right']['z']}"
-      roll="${calibration['top_unit_base_link2gnss_right']['roll']}"
-      pitch="${calibration['top_unit_base_link2gnss_right']['pitch']}"
-      yaw="${calibration['top_unit_base_link2gnss_right']['yaw']}"
-      fps="100" />
+      x="${calibration['top_unit_base_link']['gnss_right']['x']}"
+      y="${calibration['top_unit_base_link']['gnss_right']['y']}"
+      z="${calibration['top_unit_base_link']['gnss_right']['z']}"
+      roll="${calibration['top_unit_base_link']['gnss_right']['roll']}"
+      pitch="${calibration['top_unit_base_link']['gnss_right']['pitch']}"
+      yaw="${calibration['top_unit_base_link']['gnss_right']['yaw']}"
+      fps="100"
+    />
     <!-- right -->
     <xacro:imu_macro
@@ -83,11 +180,12 @@
       parent="top_unit_base_link"
       namespace=""
-      x="${calibration['top_unit_base_link2gnss_left']['x']}"
-      y="${calibration['top_unit_base_link2gnss_left']['y']}"
-      z="${calibration['top_unit_base_link2gnss_left']['z']}"
-      roll="${calibration['top_unit_base_link2gnss_left']['roll']}"
-      pitch="${calibration['top_unit_base_link2gnss_left']['pitch']}"
-      yaw="${calibration['top_unit_base_link2gnss_left']['yaw']}"
-      fps="100" />
+      x="${calibration['top_unit_base_link']['gnss_left']['x']}"
+      y="${calibration['top_unit_base_link']['gnss_left']['y']}"
+      z="${calibration['top_unit_base_link']['gnss_left']['z']}"
+      roll="${calibration['top_unit_base_link']['gnss_left']['roll']}"
+      pitch="${calibration['top_unit_base_link']['gnss_left']['pitch']}"
+      yaw="${calibration['top_unit_base_link']['gnss_left']['yaw']}"
+      fps="100"
+    />
     <!-- imu -->
     <xacro:imu_macro
@@ -95,11 +193,12 @@
       parent="top_unit_base_link"
       namespace=""
-      x="${calibration['top_unit_base_link2imu_tamagawa']['x']}"
-      y="${calibration['top_unit_base_link2imu_tamagawa']['y']}"
-      z="${calibration['top_unit_base_link2imu_tamagawa']['z']}"
-      roll="${calibration['top_unit_base_link2imu_tamagawa']['roll']}"
-      pitch="${calibration['top_unit_base_link2imu_tamagawa']['pitch']}"
-      yaw="${calibration['top_unit_base_link2imu_tamagawa']['yaw']}"
-      fps="100" />
+      x="${calibration['top_unit_base_link']['imu_tamagawa']['x']}"
+      y="${calibration['top_unit_base_link']['imu_tamagawa']['y']}"
+      z="${calibration['top_unit_base_link']['imu_tamagawa']['z']}"
+      roll="${calibration['top_unit_base_link']['imu_tamagawa']['roll']}"
+      pitch="${calibration['top_unit_base_link']['imu_tamagawa']['pitch']}"
+      yaw="${calibration['top_unit_base_link']['imu_tamagawa']['yaw']}"
+      fps="100"
+    />
   </xacro:macro>
 </robot>
