Commit message: add xacro:if to aip_xx1_description

File: aip_xx1_description/urdf/sensor_kit.xacro (robot description, xacro)
@@ -21,203 +21,230 @@
     <!-- sensor -->
     <xacro:property name="calibration" value="${load_yaml('$(arg config_dir)/sensor_kit_calibration.yaml')}"/>
-    <!-- lidar -->
-    <xacro:VLS-128
-      parent="sensor_kit_base_link"
-      name="velodyne_top"
-      topic="/points_raw"
-      hz="10"
-      samples="220"
-      gpu="$(arg gpu)"
-    >
-      <origin
-        xyz="${calibration['sensor_kit_base_link']['velodyne_top_base_link']['x']}
-             ${calibration['sensor_kit_base_link']['velodyne_top_base_link']['y']}
-             ${calibration['sensor_kit_base_link']['velodyne_top_base_link']['z']}"
-        rpy="${calibration['sensor_kit_base_link']['velodyne_top_base_link']['roll']}
-             ${calibration['sensor_kit_base_link']['velodyne_top_base_link']['pitch']}
-             ${calibration['sensor_kit_base_link']['velodyne_top_base_link']['yaw']}"
-      />
-    </xacro:VLS-128>
-    <xacro:VLP-16
-      parent="sensor_kit_base_link"
-      name="velodyne_left"
-      topic="/points_raw"
-      hz="10"
-      samples="220"
-      gpu="$(arg gpu)"
-    >
-      <origin
-        xyz="${calibration['sensor_kit_base_link']['velodyne_left_base_link']['x']}
-             ${calibration['sensor_kit_base_link']['velodyne_left_base_link']['y']}
-             ${calibration['sensor_kit_base_link']['velodyne_left_base_link']['z']}"
-        rpy="${calibration['sensor_kit_base_link']['velodyne_left_base_link']['roll']}
-             ${calibration['sensor_kit_base_link']['velodyne_left_base_link']['pitch']}
-             ${calibration['sensor_kit_base_link']['velodyne_left_base_link']['yaw']}"
-      />
-    </xacro:VLP-16>
-    <xacro:VLP-16
-      parent="sensor_kit_base_link"
-      name="velodyne_right"
-      topic="/points_raw"
-      hz="10"
-      samples="220"
-      gpu="$(arg gpu)"
-    >
-      <origin
-        xyz="${calibration['sensor_kit_base_link']['velodyne_right_base_link']['x']}
-             ${calibration['sensor_kit_base_link']['velodyne_right_base_link']['y']}
-             ${calibration['sensor_kit_base_link']['velodyne_right_base_link']['z']}"
-        rpy="${calibration['sensor_kit_base_link']['velodyne_right_base_link']['roll']}
-             ${calibration['sensor_kit_base_link']['velodyne_right_base_link']['pitch']}
-             ${calibration['sensor_kit_base_link']['velodyne_right_base_link']['yaw']}"
-      />
-    </xacro:VLP-16>
+    <xacro:property name="available_sensors" value="${calibration['sensor_kit_base_link']}"/>
+       <!-- lidar -->
+    <xacro:if value="${'velodyne_top_base_link' in available_sensors}">
+      <xacro:VLS-128
+        parent="sensor_kit_base_link"
+        name="velodyne_top"
+        topic="/points_raw"
+        hz="10"
+        samples="220"
+        gpu="$(arg gpu)"
+      >
+        <origin
+          xyz="${calibration['sensor_kit_base_link']['velodyne_top_base_link']['x']}
+               ${calibration['sensor_kit_base_link']['velodyne_top_base_link']['y']}
+               ${calibration['sensor_kit_base_link']['velodyne_top_base_link']['z']}"
+          rpy="${calibration['sensor_kit_base_link']['velodyne_top_base_link']['roll']}
+               ${calibration['sensor_kit_base_link']['velodyne_top_base_link']['pitch']}
+               ${calibration['sensor_kit_base_link']['velodyne_top_base_link']['yaw']}"
+        />
+      </xacro:VLS-128>
+    </xacro:if>
+    <xacro:if value="${'velodyne_left_base_link' in available_sensors}">
+      <xacro:VLP-16
+        parent="sensor_kit_base_link"
+        name="velodyne_left"
+        topic="/points_raw"
+        hz="10"
+        samples="220"
+        gpu="$(arg gpu)"
+      >
+        <origin
+          xyz="${calibration['sensor_kit_base_link']['velodyne_left_base_link']['x']}
+               ${calibration['sensor_kit_base_link']['velodyne_left_base_link']['y']}
+               ${calibration['sensor_kit_base_link']['velodyne_left_base_link']['z']}"
+          rpy="${calibration['sensor_kit_base_link']['velodyne_left_base_link']['roll']}
+               ${calibration['sensor_kit_base_link']['velodyne_left_base_link']['pitch']}
+               ${calibration['sensor_kit_base_link']['velodyne_left_base_link']['yaw']}"
+        />
+      </xacro:VLP-16>
+    </xacro:if>
+    <xacro:if value="${'velodyne_right_base_link' in available_sensors}">
+      <xacro:VLP-16
+        parent="sensor_kit_base_link"
+        name="velodyne_right"
+        topic="/points_raw"
+        hz="10"
+        samples="220"
+        gpu="$(arg gpu)"
+      >
+        <origin
+          xyz="${calibration['sensor_kit_base_link']['velodyne_right_base_link']['x']}
+               ${calibration['sensor_kit_base_link']['velodyne_right_base_link']['y']}
+               ${calibration['sensor_kit_base_link']['velodyne_right_base_link']['z']}"
+          rpy="${calibration['sensor_kit_base_link']['velodyne_right_base_link']['roll']}
+               ${calibration['sensor_kit_base_link']['velodyne_right_base_link']['pitch']}
+               ${calibration['sensor_kit_base_link']['velodyne_right_base_link']['yaw']}"
+        />
+      </xacro:VLP-16>
+    </xacro:if>
     <!-- camera -->
-    <xacro:monocular_camera_macro
-      name="traffic_light_right_camera/camera"
-      parent="sensor_kit_base_link"
-      namespace=""
-      x="${calibration['sensor_kit_base_link']['traffic_light_right_camera/camera_link']['x']}"
-      y="${calibration['sensor_kit_base_link']['traffic_light_right_camera/camera_link']['y']}"
-      z="${calibration['sensor_kit_base_link']['traffic_light_right_camera/camera_link']['z']}"
-      roll="${calibration['sensor_kit_base_link']['traffic_light_right_camera/camera_link']['roll']}"
-      pitch="${calibration['sensor_kit_base_link']['traffic_light_right_camera/camera_link']['pitch']}"
-      yaw="${calibration['sensor_kit_base_link']['traffic_light_right_camera/camera_link']['yaw']}"
-      fps="30"
-      width="800"
-      height="400"
-      fov="1.3"
-    />
-    <xacro:monocular_camera_macro
-      name="traffic_light_left_camera/camera"
-      parent="sensor_kit_base_link"
-      namespace=""
-      x="${calibration['sensor_kit_base_link']['traffic_light_left_camera/camera_link']['x']}"
-      y="${calibration['sensor_kit_base_link']['traffic_light_left_camera/camera_link']['y']}"
-      z="${calibration['sensor_kit_base_link']['traffic_light_left_camera/camera_link']['z']}"
-      roll="${calibration['sensor_kit_base_link']['traffic_light_left_camera/camera_link']['roll']}"
-      pitch="${calibration['sensor_kit_base_link']['traffic_light_left_camera/camera_link']['pitch']}"
-      yaw="${calibration['sensor_kit_base_link']['traffic_light_left_camera/camera_link']['yaw']}"
-      fps="30"
-      width="800"
-      height="400"
-      fov="1.3"
-    />
-    <xacro:monocular_camera_macro
-      name="camera0/camera"
-      parent="sensor_kit_base_link"
-      namespace=""
-      x="${calibration['sensor_kit_base_link']['camera0/camera_link']['x']}"
-      y="${calibration['sensor_kit_base_link']['camera0/camera_link']['y']}"
-      z="${calibration['sensor_kit_base_link']['camera0/camera_link']['z']}"
-      roll="${calibration['sensor_kit_base_link']['camera0/camera_link']['roll']}"
-      pitch="${calibration['sensor_kit_base_link']['camera0/camera_link']['pitch']}"
-      yaw="${calibration['sensor_kit_base_link']['camera0/camera_link']['yaw']}"
-      fps="30"
-      width="800"
-      height="400"
-      fov="1.3"
-    />
-    <xacro:monocular_camera_macro
-      name="camera1/camera"
-      parent="sensor_kit_base_link"
-      namespace=""
-      x="${calibration['sensor_kit_base_link']['camera1/camera_link']['x']}"
-      y="${calibration['sensor_kit_base_link']['camera1/camera_link']['y']}"
-      z="${calibration['sensor_kit_base_link']['camera1/camera_link']['z']}"
-      roll="${calibration['sensor_kit_base_link']['camera1/camera_link']['roll']}"
-      pitch="${calibration['sensor_kit_base_link']['camera1/camera_link']['pitch']}"
-      yaw="${calibration['sensor_kit_base_link']['camera1/camera_link']['yaw']}"
-      fps="30"
-      width="800"
-      height="400"
-      fov="1.3"
-    />
-    <xacro:monocular_camera_macro
-      name="camera2/camera"
-      parent="sensor_kit_base_link"
-      namespace=""
-      x="${calibration['sensor_kit_base_link']['camera2/camera_link']['x']}"
-      y="${calibration['sensor_kit_base_link']['camera2/camera_link']['y']}"
-      z="${calibration['sensor_kit_base_link']['camera2/camera_link']['z']}"
-      roll="${calibration['sensor_kit_base_link']['camera2/camera_link']['roll']}"
-      pitch="${calibration['sensor_kit_base_link']['camera2/camera_link']['pitch']}"
-      yaw="${calibration['sensor_kit_base_link']['camera2/camera_link']['yaw']}"
-      fps="30"
-      width="800"
-      height="400"
-      fov="1.3"
-    />
-    <xacro:monocular_camera_macro
-      name="camera3/camera"
-      parent="sensor_kit_base_link"
-      namespace=""
-      x="${calibration['sensor_kit_base_link']['camera3/camera_link']['x']}"
-      y="${calibration['sensor_kit_base_link']['camera3/camera_link']['y']}"
-      z="${calibration['sensor_kit_base_link']['camera3/camera_link']['z']}"
-      roll="${calibration['sensor_kit_base_link']['camera3/camera_link']['roll']}"
-      pitch="${calibration['sensor_kit_base_link']['camera3/camera_link']['pitch']}"
-      yaw="${calibration['sensor_kit_base_link']['camera3/camera_link']['yaw']}"
-      fps="30"
-      width="800"
-      height="400"
-      fov="1.3"
-    />
-    <xacro:monocular_camera_macro
-      name="camera4/camera"
-      parent="sensor_kit_base_link"
-      namespace=""
-      x="${calibration['sensor_kit_base_link']['camera4/camera_link']['x']}"
-      y="${calibration['sensor_kit_base_link']['camera4/camera_link']['y']}"
-      z="${calibration['sensor_kit_base_link']['camera4/camera_link']['z']}"
-      roll="${calibration['sensor_kit_base_link']['camera4/camera_link']['roll']}"
-      pitch="${calibration['sensor_kit_base_link']['camera4/camera_link']['pitch']}"
-      yaw="${calibration['sensor_kit_base_link']['camera4/camera_link']['yaw']}"
-      fps="30"
-      width="800"
-      height="400"
-      fov="1.3"
-    />
-    <xacro:monocular_camera_macro
-      name="camera5/camera"
-      parent="sensor_kit_base_link"
-      namespace=""
-      x="${calibration['sensor_kit_base_link']['camera5/camera_link']['x']}"
-      y="${calibration['sensor_kit_base_link']['camera5/camera_link']['y']}"
-      z="${calibration['sensor_kit_base_link']['camera5/camera_link']['z']}"
-      roll="${calibration['sensor_kit_base_link']['camera5/camera_link']['roll']}"
-      pitch="${calibration['sensor_kit_base_link']['camera5/camera_link']['pitch']}"
-      yaw="${calibration['sensor_kit_base_link']['camera5/camera_link']['yaw']}"
-      fps="30"
-      width="800"
-      height="400"
-      fov="1.3"
-    />
+    <xacro:if value="${'traffic_light_right_camera/camera_link' in available_sensors}">
+      <xacro:monocular_camera_macro
+        name="traffic_light_right_camera/camera"
+        parent="sensor_kit_base_link"
+        namespace=""
+        x="${calibration['sensor_kit_base_link']['traffic_light_right_camera/camera_link']['x']}"
+        y="${calibration['sensor_kit_base_link']['traffic_light_right_camera/camera_link']['y']}"
+        z="${calibration['sensor_kit_base_link']['traffic_light_right_camera/camera_link']['z']}"
+        roll="${calibration['sensor_kit_base_link']['traffic_light_right_camera/camera_link']['roll']}"
+        pitch="${calibration['sensor_kit_base_link']['traffic_light_right_camera/camera_link']['pitch']}"
+        yaw="${calibration['sensor_kit_base_link']['traffic_light_right_camera/camera_link']['yaw']}"
+        fps="30"
+        width="800"
+        height="400"
+        fov="1.3"
+      />
+    </xacro:if>
+    <xacro:if value="${'traffic_light_left_camera/camera_link' in available_sensors}">
+      <xacro:monocular_camera_macro
+        name="traffic_light_left_camera/camera"
+        parent="sensor_kit_base_link"
+        namespace=""
+        x="${calibration['sensor_kit_base_link']['traffic_light_left_camera/camera_link']['x']}"
+        y="${calibration['sensor_kit_base_link']['traffic_light_left_camera/camera_link']['y']}"
+        z="${calibration['sensor_kit_base_link']['traffic_light_left_camera/camera_link']['z']}"
+        roll="${calibration['sensor_kit_base_link']['traffic_light_left_camera/camera_link']['roll']}"
+        pitch="${calibration['sensor_kit_base_link']['traffic_light_left_camera/camera_link']['pitch']}"
+        yaw="${calibration['sensor_kit_base_link']['traffic_light_left_camera/camera_link']['yaw']}"
+        fps="30"
+        width="800"
+        height="400"
+        fov="1.3"
+      />
+    </xacro:if>
+    <xacro:if value="${'camera0/camera_link' in available_sensors}">
+      <xacro:monocular_camera_macro
+        name="camera0/camera"
+        parent="sensor_kit_base_link"
+        namespace=""
+        x="${calibration['sensor_kit_base_link']['camera0/camera_link']['x']}"
+        y="${calibration['sensor_kit_base_link']['camera0/camera_link']['y']}"
+        z="${calibration['sensor_kit_base_link']['camera0/camera_link']['z']}"
+        roll="${calibration['sensor_kit_base_link']['camera0/camera_link']['roll']}"
+        pitch="${calibration['sensor_kit_base_link']['camera0/camera_link']['pitch']}"
+        yaw="${calibration['sensor_kit_base_link']['camera0/camera_link']['yaw']}"
+        fps="30"
+        width="800"
+        height="400"
+        fov="1.3"
+      />
+    </xacro:if>
+    <xacro:if value="${'camera1/camera_link' in available_sensors}">
+      <xacro:monocular_camera_macro
+        name="camera1/camera"
+        parent="sensor_kit_base_link"
+        namespace=""
+        x="${calibration['sensor_kit_base_link']['camera1/camera_link']['x']}"
+        y="${calibration['sensor_kit_base_link']['camera1/camera_link']['y']}"
+        z="${calibration['sensor_kit_base_link']['camera1/camera_link']['z']}"
+        roll="${calibration['sensor_kit_base_link']['camera1/camera_link']['roll']}"
+        pitch="${calibration['sensor_kit_base_link']['camera1/camera_link']['pitch']}"
+        yaw="${calibration['sensor_kit_base_link']['camera1/camera_link']['yaw']}"
+        fps="30"
+        width="800"
+        height="400"
+        fov="1.3"
+      />
+    </xacro:if>
+    <xacro:if value="${'camera2/camera_link' in available_sensors}">
+      <xacro:monocular_camera_macro
+        name="camera2/camera"
+        parent="sensor_kit_base_link"
+        namespace=""
+        x="${calibration['sensor_kit_base_link']['camera2/camera_link']['x']}"
+        y="${calibration['sensor_kit_base_link']['camera2/camera_link']['y']}"
+        z="${calibration['sensor_kit_base_link']['camera2/camera_link']['z']}"
+        roll="${calibration['sensor_kit_base_link']['camera2/camera_link']['roll']}"
+        pitch="${calibration['sensor_kit_base_link']['camera2/camera_link']['pitch']}"
+        yaw="${calibration['sensor_kit_base_link']['camera2/camera_link']['yaw']}"
+        fps="30"
+        width="800"
+        height="400"
+        fov="1.3"
+      />
+    </xacro:if>
+    <xacro:if value="${'camera3/camera_link' in available_sensors}">
+      <xacro:monocular_camera_macro
+        name="camera3/camera"
+        parent="sensor_kit_base_link"
+        namespace=""
+        x="${calibration['sensor_kit_base_link']['camera3/camera_link']['x']}"
+        y="${calibration['sensor_kit_base_link']['camera3/camera_link']['y']}"
+        z="${calibration['sensor_kit_base_link']['camera3/camera_link']['z']}"
+        roll="${calibration['sensor_kit_base_link']['camera3/camera_link']['roll']}"
+        pitch="${calibration['sensor_kit_base_link']['camera3/camera_link']['pitch']}"
+        yaw="${calibration['sensor_kit_base_link']['camera3/camera_link']['yaw']}"
+        fps="30"
+        width="800"
+        height="400"
+        fov="1.3"
+      />
+    </xacro:if>
+    <xacro:if value="${'camera4/camera_link' in available_sensors}">
+      <xacro:monocular_camera_macro
+        name="camera4/camera"
+        parent="sensor_kit_base_link"
+        namespace=""
+        x="${calibration['sensor_kit_base_link']['camera4/camera_link']['x']}"
+        y="${calibration['sensor_kit_base_link']['camera4/camera_link']['y']}"
+        z="${calibration['sensor_kit_base_link']['camera4/camera_link']['z']}"
+        roll="${calibration['sensor_kit_base_link']['camera4/camera_link']['roll']}"
+        pitch="${calibration['sensor_kit_base_link']['camera4/camera_link']['pitch']}"
+        yaw="${calibration['sensor_kit_base_link']['camera4/camera_link']['yaw']}"
+        fps="30"
+        width="800"
+        height="400"
+        fov="1.3"
+      />
+    </xacro:if>
+    <xacro:if value="${'camera5/camera_link' in available_sensors}">
+      <xacro:monocular_camera_macro
+        name="camera5/camera"
+        parent="sensor_kit_base_link"
+        namespace=""
+        x="${calibration['sensor_kit_base_link']['camera5/camera_link']['x']}"
+        y="${calibration['sensor_kit_base_link']['camera5/camera_link']['y']}"
+        z="${calibration['sensor_kit_base_link']['camera5/camera_link']['z']}"
+        roll="${calibration['sensor_kit_base_link']['camera5/camera_link']['roll']}"
+        pitch="${calibration['sensor_kit_base_link']['camera5/camera_link']['pitch']}"
+        yaw="${calibration['sensor_kit_base_link']['camera5/camera_link']['yaw']}"
+        fps="30"
+        width="800"
+        height="400"
+        fov="1.3"
+      />
+    </xacro:if>
     <!-- gnss -->
-    <xacro:imu_macro
-      name="gnss"
-      parent="sensor_kit_base_link"
-      namespace=""
-      x="${calibration['sensor_kit_base_link']['gnss_link']['x']}"
-      y="${calibration['sensor_kit_base_link']['gnss_link']['y']}"
-      z="${calibration['sensor_kit_base_link']['gnss_link']['z']}"
-      roll="${calibration['sensor_kit_base_link']['gnss_link']['roll']}"
-      pitch="${calibration['sensor_kit_base_link']['gnss_link']['pitch']}"
-      yaw="${calibration['sensor_kit_base_link']['gnss_link']['yaw']}"
-      fps="100"
-    />
+    <xacro:if value="${'gnss_link' in available_sensors}">
+      <xacro:imu_macro
+        name="gnss"
+        parent="sensor_kit_base_link"
+        namespace=""
+        x="${calibration['sensor_kit_base_link']['gnss_link']['x']}"
+        y="${calibration['sensor_kit_base_link']['gnss_link']['y']}"
+        z="${calibration['sensor_kit_base_link']['gnss_link']['z']}"
+        roll="${calibration['sensor_kit_base_link']['gnss_link']['roll']}"
+        pitch="${calibration['sensor_kit_base_link']['gnss_link']['pitch']}"
+        yaw="${calibration['sensor_kit_base_link']['gnss_link']['yaw']}"
+        fps="100"
+      />
+    </xacro:if>
     <!-- imu -->
-    <xacro:imu_macro
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